File: BBB_LEA-M8T_CAPE.brd (EAGLE design)
At the start: 54.6 x 71.8 mm, 36 parts, among them U2 MIC5225-3.3

Commit message: added eeprom to ublox LEA cape
Parts:
- added C19: 0.1uF, microbuilder:0805-NO
- added C20: 10uF, microbuilder:0805-NO
- added R6: 10K, microbuilder:0805-NO
- added S1: DIP-02-SMD-50MIL, SparkFun-Switches:DIPSWITCH-02-50MIL
- added U1: 24LC256, SparkFun-IC-Memory:SO08
Connections:
- new net I2C2_SCL: U$15.65
- new net I2C2_SDA: U$15.66
- new net N$13: R6.2, U1.3
- new net N$15: S1.3, U1.2
- new net N$16: S1.4, U1.1
- net 3.3V: now also C19.1, C20.1, R6.1, U1.8
- net GND: now also C19.2, C20.2, S1.1, S1.2, U1.4
- net SCL: now also U1.6
- net SDA: now also U1.5
Routing:
- net GND: track 59.2 -> 67.6 mm, vias 19 -> 23
- net SDA: track 28.6 -> 34.3 mm, vias 0 -> 2
- net SCL: track 34.5 -> 38.0 mm
- net N$13: track 0.00 -> 2.97 mm
- net N$16: track 0.00 -> 1.88 mm
- net N$15: track 0.00 -> 1.88 mm
Changed lines of the file:
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@@
 <text x="49.022" y="6.096" size="0.635" layer="25">4
   3</text>
-<wire x1="13.97" y1="39.116" x2="13.97" y2="38.1" width="0.4064" layer="20"/>
-<wire x1="13.97" y1="37.084" x2="13.97" y2="36.068" width="0.4064" layer="20"/>
-<wire x1="21.59" y1="37.084" x2="21.59" y2="36.068" width="0.4064" layer="20"/>
-<wire x1="21.59" y1="35.306" x2="21.59" y2="34.29" width="0.4064" layer="20"/>
-<wire x1="26.67" y1="33.274" x2="26.67" y2="32.258" width="0.4064" layer="20"/>
-<wire x1="26.67" y1="31.496" x2="26.67" y2="30.48" width="0.4064" layer="20"/>
+<wire x1="13.97" y1="39.116" x2="13.97" y2="38.1" width="0.4064" layer="25"/>
+<wire x1="13.97" y1="37.084" x2="13.97" y2="36.068" width="0.4064" layer="25"/>
+<wire x1="21.59" y1="37.084" x2="21.59" y2="36.068" width="0.4064" layer="25"/>
+<wire x1="21.59" y1="35.306" x2="21.59" y2="34.29" width="0.4064" layer="25"/>
+<wire x1="26.67" y1="33.274" x2="26.67" y2="32.258" width="0.4064" layer="25"/>
+<wire x1="26.67" y1="31.496" x2="26.67" y2="30.48" width="0.4064" layer="25"/>
 </plain>
 <attributes>
@@
 <attribute name="NAME" x="37.338" y="18.415" size="0.635" layer="25"/>
 </element>
+<element name="U1" library="SparkFun-IC-Memory" package="SO08" value="24LC256" x="37.084" y="39.878" smashed="yes" rot="R180">
+<attribute name="PROD_ID" value="IC-09714" x="37.084" y="39.878" size="1.778" layer="27" rot="R180" display="off"/>
+<attribute name="VALUE" x="36.83" y="39.624" size="0.6096" layer="27" font="vector" ratio="20" align="bottom-center"/>
+</element>
+<element name="S1" library="SparkFun-Switches" package="DIPSWITCH-02-50MIL" value="DIP-02-SMD-50MIL" x="38.354" y="48.26" smashed="yes" rot="R180">
+<attribute name="PROD_ID" value="SWCH-13215" x="38.354" y="48.26" size="1.778" layer="27" rot="R180" display="off"/>
+<attribute name="NAME" x="40.513" y="48.26" size="0.6096" layer="25" font="vector" ratio="20" rot="R270" align="bottom-center"/>
+</element>
+<element name="R6" library="microbuilder" package="0805-NO" value="10K" x="34.036" y="44.704" smashed="yes">
+<attribute name="NAME" x="33.528" y="45.847" size="0.635" layer="25"/>
+</element>
+<element name="C19" library="microbuilder" package="0805-NO" value="0.1uF" x="41.402" y="36.068" smashed="yes" rot="R270">
+<attribute name="NAME" x="39.751" y="35.56" size="0.635" layer="25" rot="R270"/>
+</element>
+<element name="C20" library="microbuilder" package="0805-NO" value="10uF" x="41.402" y="39.878" smashed="yes" rot="R90">
+<attribute name="NAME" x="40.64" y="41.783" size="0.635" layer="25"/>
+</element>
 </elements>
 <signals>
@@
 <wire x1="15.272" y1="28.466" x2="14.968" y2="28.466" width="0.4064" layer="1"/>
 <wire x1="14.968" y1="28.466" x2="13.97" y2="28.448" width="0.4064" layer="1"/>
+<contactref element="S1" pad="1"/>
+<contactref element="S1" pad="2"/>
+<contactref element="U1" pad="4"/>
+<contactref element="C19" pad="2"/>
+<contactref element="C20" pad="2"/>
+<via x="41.402" y="43.18" extent="1-16" drill="0.6" shape="square"/>
+<via x="42.164" y="33.782" extent="1-16" drill="0.6" shape="square"/>
+<wire x1="41.402" y1="35.118" x2="41.402" y2="34.544" width="0.4064" layer="1"/>
+<wire x1="41.402" y1="34.544" x2="42.164" y2="33.782" width="0.4064" layer="1"/>
+<wire x1="41.402" y1="40.828" x2="41.402" y2="43.18" width="0.4064" layer="1"/>
+<via x="33.782" y="42.672" extent="1-16" drill="0.6" shape="square"/>
+<wire x1="33.782" y1="42.672" x2="35.173" y2="42.672" width="0.4064" layer="1"/>
+<wire x1="35.173" y1="42.672" x2="35.179" y2="42.678" width="0.4064" layer="1"/>
+<via x="38.354" y="53.594" extent="1-16" drill="0.6" shape="square"/>
+<wire x1="37.719" y1="51.96" x2="38.354" y2="51.96" width="0.4064" layer="1"/>
+<wire x1="38.354" y1="51.96" x2="38.989" y2="51.96" width="0.4064" layer="1"/>
+<wire x1="38.354" y1="53.594" x2="38.354" y2="51.96" width="0.4064" layer="1"/>
 </signal>
 <signal name="3.3V">
@@
 <wire x1="32.512" y1="30.734" x2="32.512" y2="34.544" width="0.4064" layer="16"/>
 <wire x1="32.512" y1="34.544" x2="32.766" y2="34.798" width="0.4064" layer="16"/>
+<contactref element="R6" pad="1"/>
+<contactref element="C19" pad="1"/>
+<contactref element="C20" pad="1"/>
+<contactref element="U1" pad="8"/>
 </signal>
 <signal name="ENABLE">
@@
 <contactref element="U$1" pad="28"/>
 <wire x1="32.272" y1="11.666" x2="32.272" y2="13.956" width="0.4064" layer="1"/>
-<wire x1="32.272" y1="13.956" x2="29.972" y2="16.256" width="0.4064" layer="1"/>
-<wire x1="29.972" y1="16.256" x2="12.192" y2="16.256" width="0.4064" layer="1"/>
-<wire x1="12.192" y1="16.256" x2="8.382" y2="12.192" width="0.4064" layer="1"/>
+<wire x1="32.272" y1="13.956" x2="29.718" y2="16.51" width="0.4064" layer="1"/>
+<wire x1="29.718" y1="16.51" x2="12.446" y2="16.51" width="0.4064" layer="1"/>
+<wire x1="12.446" y1="16.51" x2="8.382" y2="12.192" width="0.4064" layer="1"/>
 <wire x1="8.382" y1="12.192" x2="7.239" y2="12.192" width="0.4064" layer="1"/>
 </signal>
@@
 <wire x1="32.272" y1="28.466" x2="32.342" y2="28.466" width="0.4064" layer="1"/>
 <wire x1="32.342" y1="28.466" x2="34.61" y2="30.734" width="0.4064" layer="1"/>
-<wire x1="34.61" y1="30.734" x2="34.61" y2="31.562" width="0.4064" layer="1"/>
-<wire x1="34.61" y1="31.562" x2="35.56" y2="32.512" width="0.4064" layer="1"/>
-<wire x1="35.56" y1="32.512" x2="39.116" y2="32.512" width="0.4064" layer="1"/>
-<wire x1="39.116" y1="32.512" x2="43.18" y2="28.448" width="0.4064" layer="1"/>
+<wire x1="37.846" y1="32.258" x2="39.37" y2="32.258" width="0.4064" layer="1"/>
+<wire x1="39.37" y1="32.258" x2="43.18" y2="28.448" width="0.4064" layer="1"/>
 <wire x1="43.18" y1="28.448" x2="43.18" y2="25.4" width="0.4064" layer="1"/>
 <wire x1="43.18" y1="25.4" x2="44.704" y2="23.876" width="0.4064" layer="1"/>
 <wire x1="44.704" y1="23.876" x2="47.3964" y2="23.876" width="0.4064" layer="1"/>
 <wire x1="47.3964" y1="23.876" x2="47.5234" y2="24.003" width="0.4064" layer="1"/>
+<contactref element="U1" pad="5"/>
+<via x="37.846" y="32.258" extent="1-16" drill="0.6" shape="square"/>
+<wire x1="37.846" y1="32.258" x2="35.56" y2="34.798" width="0.4064" layer="16"/>
+<wire x1="35.56" y1="34.798" x2="35.306" y2="35.052" width="0.4064" layer="16"/>
+<via x="35.306" y="35.052" extent="1-16" drill="0.6" shape="square"/>
+<wire x1="35.306" y1="35.052" x2="35.179" y2="35.179" width="0.4064" layer="1"/>
+<wire x1="35.179" y1="35.179" x2="35.179" y2="37.078" width="0.4064" layer="1"/>
+<wire x1="37.846" y1="32.258" x2="35.306" y2="32.258" width="0.4064" layer="1"/>
+<wire x1="35.306" y1="32.258" x2="34.544" y2="31.496" width="0.4064" layer="1"/>
+<wire x1="34.544" y1="31.496" x2="34.544" y2="30.8" width="0.4064" layer="1"/>
+<wire x1="34.544" y1="30.8" x2="34.61" y2="30.734" width="0.4064" layer="1"/>
 </signal>
 <signal name="SCL">
@@
 <wire x1="44.704" y1="26.162" x2="44.704" y2="28.956" width="0.4064" layer="1"/>
 <wire x1="44.704" y1="28.956" x2="39.878" y2="33.782" width="0.4064" layer="1"/>
-<wire x1="39.878" y1="33.782" x2="34.544" y2="33.782" width="0.4064" layer="1"/>
+<wire x1="39.878" y1="33.782" x2="36.322" y2="33.782" width="0.4064" layer="1"/>
+<wire x1="36.322" y1="33.782" x2="34.544" y2="33.782" width="0.4064" layer="1"/>
 <wire x1="34.544" y1="33.782" x2="32.512" y2="31.75" width="0.4064" layer="1"/>
 <wire x1="32.512" y1="31.75" x2="31.816" y2="31.75" width="0.4064" layer="1"/>
 <wire x1="31.816" y1="31.75" x2="30.988" y2="31.562" width="0.4064" layer="1"/>
+<contactref element="U1" pad="6"/>
+<wire x1="36.449" y1="37.078" x2="36.322" y2="37.078" width="0.4064" layer="1"/>
+<wire x1="36.322" y1="37.078" x2="36.322" y2="33.782" width="0.4064" layer="1"/>
 </signal>
 <signal name="SQW">
@@
 <contactref element="U$15" pad="5"/>
 <wire x1="31.172" y1="11.666" x2="31.172" y2="13.024" width="0.4064" layer="1"/>
-<wire x1="31.172" y1="13.024" x2="29.21" y2="14.986" width="0.4064" layer="1"/>
-<wire x1="29.21" y1="14.986" x2="13.97" y2="14.986" width="0.4064" layer="1"/>
-<wire x1="13.97" y1="14.986" x2="8.636" y2="9.652" width="0.4064" layer="1"/>
+<wire x1="31.172" y1="13.024" x2="28.956" y2="15.24" width="0.4064" layer="1"/>
+<wire x1="28.956" y1="15.24" x2="14.224" y2="15.24" width="0.4064" layer="1"/>
+<wire x1="14.224" y1="15.24" x2="8.636" y2="9.652" width="0.4064" layer="1"/>
 <wire x1="8.636" y1="9.652" x2="7.239" y2="9.652" width="0.4064" layer="1"/>
 </signal>
@@
 <wire x1="18.756" y1="32.406" x2="18.862" y2="32.766" width="0.4064" layer="1"/>
 </signal>
+<signal name="I2C2_SCL">
+<contactref element="U$15" pad="65"/>
+</signal>
+<signal name="I2C2_SDA">
+<contactref element="U$15" pad="66"/>
+</signal>
+<signal name="N$13">
+<contactref element="U1" pad="3"/>
+<contactref element="R6" pad="2"/>
+<wire x1="36.449" y1="42.678" x2="36.449" y2="43.815" width="0.4064" layer="1"/>
+<wire x1="36.449" y1="43.815" x2="35.56" y2="44.704" width="0.4064" layer="1"/>
+<wire x1="35.56" y1="44.704" x2="34.986" y2="44.704" width="0.4064" layer="1"/>
+</signal>
+<signal name="N$15">
+<contactref element="S1" pad="3"/>
+<contactref element="U1" pad="2"/>
+<wire x1="37.719" y1="44.56" x2="37.719" y2="42.678" width="0.4064" layer="1"/>
+</signal>
+<signal name="N$16">
+<contactref element="U1" pad="1"/>
+<contactref element="S1" pad="4"/>
+<wire x1="38.989" y1="44.56" x2="38.989" y2="42.678" width="0.4064" layer="1"/>
+</signal>
 </signals>
