File: BBB_LEA-M8T_CAPE.sch (EAGLE design)
At the start: 36 parts, among them U2 MIC5225-3.3

Commit message: BOM updates associated with populating first test boards
Parts:
- C14, C7: value 22u -> 10u
- renumbered FB5 to FB4
Changed lines of the file:
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@@
 <part name="U$17" library="microbuilder" deviceset="3.3V" device=""/>
 <part name="C6" library="rcl" deviceset="C-US" device="C0805" value=".01u"/>
-<part name="C7" library="rcl" deviceset="C-US" device="C0805" value="22u"/>
+<part name="C7" library="rcl" deviceset="C-US" device="C0805" value="10u"/>
 <part name="U$21" library="microbuilder" deviceset="GND" device=""/>
 <part name="FB2" library="microbuilder" deviceset="FERRITE" device="-0805NO" value="Ferrite"/>
@@
 <part name="C12" library="microbuilder" deviceset="CAP_CERAMIC" device="0805-NOOUTLINE" value="10uF"/>
 <part name="C13" library="microbuilder" deviceset="CAP_CERAMIC" device="0805-NOOUTLINE" value="0.1uF"/>
-<part name="C14" library="rcl" deviceset="C-US" device="C0805" value="22u"/>
-<part name="FB5" library="microbuilder" deviceset="FERRITE" device="-0805NO" value="Ferrite"/>
+<part name="C14" library="rcl" deviceset="C-US" device="C0805" value="10u"/>
+<part name="FB4" library="microbuilder" deviceset="FERRITE" device="-0805NO" value="Ferrite"/>
 <part name="C15" library="microbuilder" deviceset="CAP_CERAMIC" device="0805-NOOUTLINE" value="10uF"/>
 <part name="C16" library="microbuilder" deviceset="CAP_CERAMIC" device="0805-NOOUTLINE" value="0.1uF"/>
@@
 <instance part="C13" gate="G$1" x="241.3" y="152.4" rot="MR0"/>
 <instance part="C14" gate="G$1" x="154.94" y="162.56" rot="MR270"/>
-<instance part="FB5" gate="G$1" x="172.72" y="180.34" rot="MR0"/>
+<instance part="FB4" gate="G$1" x="172.72" y="180.34" rot="MR0"/>
 <instance part="C15" gate="G$1" x="38.1" y="25.4"/>
 <instance part="C16" gate="G$1" x="45.72" y="25.4"/>
@@
 <wire x1="185.42" y1="180.34" x2="193.04" y2="180.34" width="0.1524" layer="91"/>
 <junction x="185.42" y="180.34"/>
-<pinref part="FB5" gate="G$1" pin="P$1"/>
+<pinref part="FB4" gate="G$1" pin="P$1"/>
 </segment>
 </net>
@@
 <wire x1="170.18" y1="162.56" x2="170.18" y2="170.18" width="0.1524" layer="91"/>
 <junction x="170.18" y="170.18"/>
-<pinref part="FB5" gate="G$1" pin="P$2"/>
+<pinref part="FB4" gate="G$1" pin="P$2"/>
 <junction x="170.18" y="180.34"/>
 </segment>

Commit message: added eeprom to ublox LEA cape
Parts:
- added C19: 0.1uF, microbuilder:CAP_CERAMIC0805-NOOUTLINE
- added C20: 10uF, microbuilder:CAP_CERAMIC0805-NOOUTLINE
- added R6: 10K, microbuilder:RESISTOR0805_NOOUTLINE
- added S1: DIP-02-SMD-50MIL, SparkFun-Switches:DIP-02-SMD-50MIL
- added U1: 24LC256, SparkFun-IC-Memory:EEPROM-I2CSMD
Connections:
- new net I2C2_SCL: U$15.I2C2_SCL
- new net I2C2_SDA: U$15.I2C2_SDA
- new net N$13: R6.2, U1.A2
- new net N$15: S1.P$11, U1.A1
- new net N$16: S1.P$12, U1.A0
- net 3.3V: now also C19.1, C20.1, R6.1, U1.VCC
- net GND: now also C19.2, C20.2, S1.P$1, S1.P$2, U1.VSS
- net SCL: now also U1.SCL
- net SDA: now also U1.SDA
Changed lines of the file:
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@@
 <part name="C18" library="microbuilder" deviceset="CAP_CERAMIC" device="0805-NOOUTLINE" value="0.1uF"/>
 <part name="U$11" library="microbuilder" deviceset="GND" device=""/>
+<part name="U1" library="SparkFun-IC-Memory" deviceset="EEPROM-I2C" device="SMD" value="24LC256"/>
+<part name="S1" library="SparkFun-Switches" deviceset="DIP-02" device="-SMD-50MIL"/>
+<part name="U$16" library="microbuilder" deviceset="GND" device=""/>
+<part name="R6" library="microbuilder" deviceset="RESISTOR" device="0805_NOOUTLINE" value="10K"/>
+<part name="U$18" library="microbuilder" deviceset="3.3V" device=""/>
+<part name="U$23" library="microbuilder" deviceset="GND" device=""/>
+<part name="U$25" library="microbuilder" deviceset="GND" device=""/>
+<part name="U$26" library="microbuilder" deviceset="3.3V" device=""/>
+<part name="C19" library="microbuilder" deviceset="CAP_CERAMIC" device="0805-NOOUTLINE" value="0.1uF"/>
+<part name="C20" library="microbuilder" deviceset="CAP_CERAMIC" device="0805-NOOUTLINE" value="10uF"/>
 </parts>
 <sheets>
@@
 <instance part="C18" gate="G$1" x="86.36" y="25.4"/>
 <instance part="U$11" gate="G$1" x="58.42" y="17.78" rot="MR0"/>
+<instance part="U1" gate="G$1" x="213.36" y="7.62"/>
+<instance part="S1" gate="G$1" x="165.1" y="2.54"/>
+<instance part="U$16" gate="G$1" x="165.1" y="-12.7"/>
+<instance part="R6" gate="G$1" x="177.8" y="0" rot="R90"/>
+<instance part="U$18" gate="G$1" x="177.8" y="-10.16" rot="R180"/>
+<instance part="U$23" gate="G$1" x="185.42" y="-2.54"/>
+<instance part="U$25" gate="G$1" x="256.54" y="-2.54" rot="MR0"/>
+<instance part="U$26" gate="G$1" x="264.16" y="12.7" rot="MR90"/>
+<instance part="C19" gate="G$1" x="256.54" y="7.62" rot="MR0"/>
+<instance part="C20" gate="G$1" x="248.92" y="7.62" rot="MR0"/>
 </instances>
 <busses>
@@
 <junction x="58.42" y="20.32"/>
 </segment>
+<segment>
+<pinref part="U$16" gate="G$1" pin="GND"/>
+<pinref part="S1" gate="G$1" pin="P$1"/>
+<wire x1="165.1" y1="-10.16" x2="165.1" y2="-7.62" width="0.1524" layer="91"/>
+<pinref part="S1" gate="G$1" pin="P$2"/>
+<wire x1="165.1" y1="-7.62" x2="165.1" y2="-5.08" width="0.1524" layer="91"/>
+<wire x1="167.64" y1="-5.08" x2="167.64" y2="-7.62" width="0.1524" layer="91"/>
+<wire x1="167.64" y1="-7.62" x2="165.1" y2="-7.62" width="0.1524" layer="91"/>
+<junction x="165.1" y="-7.62"/>
+</segment>
+<segment>
+<pinref part="U1" gate="G$1" pin="VSS"/>
+<wire x1="200.66" y1="5.08" x2="185.42" y2="5.08" width="0.1524" layer="91"/>
+<wire x1="185.42" y1="5.08" x2="185.42" y2="0" width="0.1524" layer="91"/>
+<pinref part="U$23" gate="G$1" pin="GND"/>
+</segment>
+<segment>
+<pinref part="U$25" gate="G$1" pin="GND"/>
+<pinref part="C19" gate="G$1" pin="2"/>
+<wire x1="256.54" y1="5.08" x2="256.54" y2="0" width="0.1524" layer="91"/>
+<junction x="256.54" y="0"/>
+<pinref part="C20" gate="G$1" pin="2"/>
+<wire x1="248.92" y1="0" x2="256.54" y2="0" width="0.1524" layer="91"/>
+<wire x1="248.92" y1="5.08" x2="248.92" y2="0" width="0.1524" layer="91"/>
+</segment>
 </net>
 <net name="3.3V" class="0">
@@
 <pinref part="FB4" gate="G$1" pin="P$1"/>
 </segment>
+<segment>
+<pinref part="R6" gate="G$1" pin="1"/>
+<pinref part="U$18" gate="G$1" pin="3.3V"/>
+<wire x1="177.8" y1="-5.08" x2="177.8" y2="-7.62" width="0.1524" layer="91"/>
+</segment>
+<segment>
+<pinref part="U$26" gate="G$1" pin="3.3V"/>
+<pinref part="C19" gate="G$1" pin="1"/>
+<junction x="261.62" y="12.7"/>
+<wire x1="248.92" y1="12.7" x2="261.62" y2="12.7" width="0.1524" layer="91"/>
+<wire x1="261.62" y1="12.7" x2="256.54" y2="12.7" width="0.1524" layer="91"/>
+<pinref part="C20" gate="G$1" pin="1"/>
+<junction x="248.92" y="12.7"/>
+<pinref part="U1" gate="G$1" pin="VCC"/>
+<wire x1="226.06" y1="12.7" x2="248.92" y2="12.7" width="0.1524" layer="91"/>
+</segment>
 </net>
 <net name="ENABLE" class="0">
@@
 <label x="220.98" y="76.2" size="1.778" layer="95"/>
 </segment>
+<segment>
+<pinref part="U1" gate="G$1" pin="SDA"/>
+<wire x1="226.06" y1="5.08" x2="241.3" y2="5.08" width="0.1524" layer="91"/>
+<label x="231.14" y="5.08" size="1.778" layer="95"/>
+</segment>
 </net>
 <net name="SCL" class="0">
@@
 <wire x1="213.36" y1="78.74" x2="226.06" y2="78.74" width="0.1524" layer="91"/>
 <label x="220.98" y="78.74" size="1.778" layer="95"/>
+</segment>
+<segment>
+<pinref part="U1" gate="G$1" pin="SCL"/>
+<wire x1="226.06" y1="7.62" x2="241.3" y2="7.62" width="0.1524" layer="91"/>
+<label x="231.14" y="7.62" size="1.778" layer="95"/>
 </segment>
 </net>
@@
 </segment>
 </net>
+<net name="I2C2_SCL" class="0">
+<segment>
+<pinref part="U$15" gate="G$1" pin="I2C2_SCL"/>
+<wire x1="22.86" y1="76.2" x2="7.62" y2="76.2" width="0.1524" layer="91"/>
+<label x="7.62" y="76.2" size="1.778" layer="95"/>
+</segment>
+</net>
+<net name="I2C2_SDA" class="0">
+<segment>
+<pinref part="U$15" gate="G$1" pin="I2C2_SDA"/>
+<wire x1="78.74" y1="76.2" x2="88.9" y2="76.2" width="0.1524" layer="91"/>
+<label x="83.82" y="76.2" size="1.778" layer="95"/>
+</segment>
+</net>
+<net name="N$13" class="0">
+<segment>
+<pinref part="U1" gate="G$1" pin="A2"/>
+<wire x1="200.66" y1="7.62" x2="177.8" y2="7.62" width="0.1524" layer="91"/>
+<wire x1="177.8" y1="7.62" x2="177.8" y2="5.08" width="0.1524" layer="91"/>
+<pinref part="R6" gate="G$1" pin="2"/>
+</segment>
+</net>
+<net name="N$15" class="0">
+<segment>
+<pinref part="S1" gate="G$1" pin="P$11"/>
+<pinref part="U1" gate="G$1" pin="A1"/>
+<wire x1="167.64" y1="10.16" x2="200.66" y2="10.16" width="0.1524" layer="91"/>
+</segment>
+</net>
+<net name="N$16" class="0">
+<segment>
+<pinref part="U1" gate="G$1" pin="A0"/>
+<pinref part="S1" gate="G$1" pin="P$12"/>
+<wire x1="200.66" y1="12.7" x2="165.1" y2="12.7" width="0.1524" layer="91"/>
+<wire x1="165.1" y1="12.7" x2="165.1" y2="10.16" width="0.1524" layer="91"/>
+</segment>
+</net>
