File: BBB_XM1100_CAPE.brd (EAGLE design)
At the start: 54.6 x 71.8 mm, 24 parts, among them U2 MIC5225-3.3

Commit message: minor layout and silkscreen cleanup
Parts:
- moved C2 1.89 mm to (34.2, 10.4), turned to 0 degrees
- moved C3 1.83 mm to (46.1, 7.75)
- moved FB1 1.32 mm to (34.2, 8.36), turned to 180 degrees
- moved R2 0.76 mm to (43.7, 9.78)
- moved C5 0.25 mm to (32.8, 12.4)
Routing:
- net VDD_5V: track 15.4 -> 13.4 mm
Changed lines of the file:
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@@
 <attribute name="NAME" x="38.735" y="8.739" size="0.4064" layer="25" ratio="15"/>
 </element>
-<element name="R2" library="microbuilder" package="0805-NO" value="10K" x="43.664" y="10.541" smashed="yes" rot="R270">
-<attribute name="NAME" x="44.934" y="11.049" size="0.635" layer="25" rot="R270"/>
-</element>
-<element name="C2" library="microbuilder" package="0805-NO" value="10uF" x="32.488" y="9.525" smashed="yes" rot="R270">
-<attribute name="NAME" x="30.559" y="9.501" size="0.635" layer="25" rot="R90"/>
-</element>
-<element name="FB1" library="microbuilder" package="0805-NO@1" value="Ferrite" x="34.774" y="9.525" smashed="yes" rot="R90">
-<attribute name="NAME" x="36.679" y="9.144" size="0.635" layer="25" rot="R90"/>
-</element>
-<element name="C3" library="microbuilder" package="0805-NO" value="10uF" x="44.553" y="6.731" smashed="yes" rot="R270">
-<attribute name="NAME" x="43.331" y="6.223" size="0.635" layer="25" rot="R90"/>
+<element name="R2" library="microbuilder" package="0805-NO" value="10K" x="43.664" y="9.779" smashed="yes" rot="R270">
+<attribute name="NAME" x="43.307" y="11.914" size="0.635" layer="25"/>
+</element>
+<element name="C2" library="microbuilder" package="0805-NO" value="10uF" x="34.163" y="10.39" smashed="yes">
+<attribute name="NAME" x="31.417" y="10.819" size="0.635" layer="25" rot="R270"/>
+</element>
+<element name="FB1" library="microbuilder" package="0805-NO@1" value="Ferrite" x="34.163" y="8.358" smashed="yes" rot="R180">
+<attribute name="NAME" x="31.647" y="9.144" size="0.635" layer="25" rot="R270"/>
+</element>
+<element name="C3" library="microbuilder" package="0805-NO" value="10uF" x="46.077" y="7.747" smashed="yes" rot="R270">
+<attribute name="NAME" x="44.855" y="6.477" size="0.635" layer="25" rot="R90"/>
 </element>
 <element name="D1" library="microbuilder" package="SOD-323" value="1N4148" x="44.704" y="18.415" smashed="yes" rot="R180">
@@
 <element name="U$3" library="tuckerLib" package="XM1100" value="XM1100" x="26.416" y="19.558" smashed="yes" rot="R90"/>
 <element name="FB2" library="microbuilder" package="0805-NO@1" value="Ferrite" x="32.766" y="16.51" smashed="yes" rot="R180">
-<attribute name="NAME" x="36.576" y="16.891" size="0.635" layer="25" rot="R180"/>
+<attribute name="NAME" x="35.179" y="17.272" size="0.635" layer="25" rot="R270"/>
 </element>
 <element name="C1" library="microbuilder" package="0805-NO" value="1.0uF" x="32.766" y="14.478" smashed="yes" rot="R180">
-<attribute name="NAME" x="36.068" y="14.859" size="0.635" layer="25" rot="R180"/>
-</element>
-<element name="C5" library="microbuilder" package="0805-NO" value="0.1uF" x="32.766" y="12.7" smashed="yes" rot="R180">
-<attribute name="NAME" x="36.068" y="13.081" size="0.635" layer="25" rot="R180"/>
+<attribute name="NAME" x="29.845" y="14.986" size="0.635" layer="25" rot="R270"/>
+</element>
+<element name="C5" library="microbuilder" package="0805-NO" value="0.1uF" x="32.766" y="12.446" smashed="yes" rot="R180">
+<attribute name="NAME" x="29.845" y="12.954" size="0.635" layer="25" rot="R270"/>
 </element>
 <element name="C6" library="microbuilder" package="0805-NO" value="1.0uF" x="32.766" y="18.542" smashed="yes">
-<attribute name="NAME" x="35.306" y="18.415" size="0.635" layer="25"/>
+<attribute name="NAME" x="35.687" y="18.034" size="0.635" layer="25" rot="R90"/>
 </element>
 <element name="C7" library="microbuilder" package="0805-NO" value="0.1uF" x="32.766" y="20.574" smashed="yes">
-<attribute name="NAME" x="35.306" y="20.447" size="0.635" layer="25"/>
+<attribute name="NAME" x="35.687" y="20.066" size="0.635" layer="25" rot="R90"/>
 </element>
 <element name="R1" library="microbuilder" package="0805-NO" value="10K" x="12.192" y="24.13" smashed="yes" rot="R270">
@@
 <via x="27.432" y="15.748" extent="1-16" drill="0.6" shape="square"/>
 <via x="27.178" y="11.43" extent="1-16" drill="0.6" shape="square"/>
-<via x="30.734" y="8.636" extent="1-16" drill="0.6" shape="square"/>
+<via x="36.576" y="11.938" extent="1-16" drill="0.6" shape="square"/>
 <via x="41.91" y="9.652" extent="1-16" drill="0.6" shape="square"/>
-<via x="46.228" y="5.842" extent="1-16" drill="0.6" shape="square"/>
-<wire x1="44.553" y1="5.781" x2="46.167" y2="5.781" width="0.4064" layer="1"/>
-<wire x1="46.167" y1="5.781" x2="46.228" y2="5.842" width="0.4064" layer="1"/>
+<via x="46.228" y="5.334" extent="1-16" drill="0.6" shape="square"/>
+<wire x1="46.077" y1="6.797" x2="46.167" y2="5.781" width="0.4064" layer="1"/>
+<wire x1="46.167" y1="5.781" x2="46.228" y2="5.334" width="0.4064" layer="1"/>
 <wire x1="40.3921" y1="9.525" x2="41.783" y2="9.525" width="0.4064" layer="1"/>
 <wire x1="41.783" y1="9.525" x2="41.91" y2="9.652" width="0.4064" layer="1"/>
-<wire x1="32.488" y1="8.575" x2="30.71" y2="8.66" width="0.4064" layer="1"/>
-<wire x1="30.71" y1="8.66" x2="30.734" y2="8.636" width="0.4064" layer="1"/>
+<wire x1="35.113" y1="10.39" x2="36.552" y2="11.708" width="0.4064" layer="1"/>
+<wire x1="36.552" y1="11.708" x2="36.576" y2="11.938" width="0.4064" layer="1"/>
 <wire x1="27.106" y1="13.138" x2="27.106" y2="11.502" width="0.4064" layer="1"/>
 <wire x1="27.106" y1="11.502" x2="27.178" y2="11.43" width="0.4064" layer="1"/>
@@
 <contactref element="C2" pad="1"/>
 <contactref element="FB1" pad="2"/>
-<wire x1="34.774" y1="10.475" x2="32.488" y2="10.475" width="0.4064" layer="1"/>
+<wire x1="33.213" y1="8.358" x2="33.213" y2="10.39" width="0.4064" layer="1"/>
 <wire x1="37.3126" y1="24.765" x2="30.353" y2="24.765" width="0.4064" layer="1"/>
 <wire x1="30.353" y1="24.765" x2="29.972" y2="24.384" width="0.4064" layer="1"/>
@@
 <contactref element="R6" pad="1"/>
 <wire x1="33.716" y1="20.574" x2="33.716" y2="18.542" width="0.4064" layer="1"/>
-<wire x1="31.816" y1="14.478" x2="31.816" y2="12.7" width="0.4064" layer="1"/>
-<wire x1="31.816" y1="12.7" x2="31.816" y2="11.147" width="0.4064" layer="1"/>
-<wire x1="31.816" y1="11.147" x2="32.488" y2="10.475" width="0.4064" layer="1"/>
+<wire x1="31.816" y1="14.478" x2="31.816" y2="12.446" width="0.4064" layer="1"/>
+<wire x1="31.816" y1="12.446" x2="31.816" y2="11.147" width="0.4064" layer="1"/>
+<wire x1="31.816" y1="11.147" x2="33.213" y2="10.39" width="0.4064" layer="1"/>
 <via x="18.542" y="14.224" extent="1-16" drill="0.6" shape="square"/>
 <wire x1="19.486" y1="11.176" x2="19.486" y2="13.28" width="0.4064" layer="1"/>
@@
 <contactref element="U2" pad="3"/>
 <contactref element="R2" pad="1"/>
-<wire x1="43.664" y1="11.491" x2="43.598" y2="11.52" width="0.4064" layer="1"/>
-<wire x1="43.598" y1="11.52" x2="43.18" y2="11.43" width="0.4064" layer="1"/>
-<wire x1="43.18" y1="11.43" x2="41.656" y2="11.43" width="0.4064" layer="1"/>
-<wire x1="41.656" y1="11.43" x2="40.64" y2="10.7229" width="0.4064" layer="1"/>
-<wire x1="40.64" y1="10.7229" x2="40.3921" y2="10.475" width="0.4064" layer="1"/>
+<wire x1="43.664" y1="10.729" x2="43.598" y2="10.758" width="0.4064" layer="1"/>
+<wire x1="43.598" y1="10.758" x2="43.434" y2="10.668" width="0.4064" layer="1"/>
+<wire x1="43.434" y1="10.668" x2="40.64" y2="10.668" width="0.4064" layer="1"/>
+<wire x1="40.64" y1="10.668" x2="40.386" y2="10.4689" width="0.4064" layer="1"/>
+<wire x1="40.386" y1="10.4689" x2="40.3921" y2="10.475" width="0.4064" layer="1"/>
 </signal>
 <signal name="N$3">
 <contactref element="FB1" pad="1"/>
 <contactref element="U2" pad="5"/>
-<wire x1="37.7919" y1="8.575" x2="34.774" y2="8.575" width="0.4064" layer="1"/>
+<wire x1="37.7919" y1="8.575" x2="35.113" y2="8.358" width="0.4064" layer="1"/>
 </signal>
 <signal name="VBACKUP">
@@
 <contactref element="C3" pad="1"/>
 <contactref element="R2" pad="2"/>
-<wire x1="52.959" y1="9.652" x2="48.006" y2="9.652" width="0.4064" layer="1"/>
-<wire x1="48.006" y1="9.652" x2="45.974" y2="7.62" width="0.4064" layer="1"/>
-<wire x1="45.974" y1="7.62" x2="44.614" y2="7.62" width="0.4064" layer="1"/>
-<wire x1="44.614" y1="7.62" x2="44.553" y2="7.681" width="0.4064" layer="1"/>
-<wire x1="44.553" y1="7.681" x2="44.389" y2="7.681" width="0.4064" layer="1"/>
-<wire x1="44.389" y1="7.681" x2="43.688" y2="8.382" width="0.4064" layer="1"/>
-<wire x1="43.307" y1="9.017" x2="43.688" y2="8.382" width="0.4064" layer="1"/>
-<wire x1="43.688" y1="8.382" x2="43.688" y2="9.483" width="0.4064" layer="1"/>
-<wire x1="43.688" y1="9.483" x2="43.664" y2="9.591" width="0.4064" layer="1"/>
+<wire x1="52.959" y1="9.652" x2="48.26" y2="9.652" width="0.4064" layer="1"/>
+<wire x1="48.26" y1="9.652" x2="46.9" y2="9.652" width="0.4064" layer="1"/>
+<wire x1="46.9" y1="9.652" x2="46.077" y2="8.697" width="0.4064" layer="1"/>
+<wire x1="46.077" y1="8.697" x2="43.881" y2="8.697" width="0.4064" layer="1"/>
+<wire x1="43.881" y1="8.697" x2="43.688" y2="8.89" width="0.4064" layer="1"/>
+<wire x1="43.561" y1="8.763" x2="43.688" y2="8.89" width="0.4064" layer="1"/>
+<wire x1="43.688" y1="8.89" x2="43.688" y2="8.975" width="0.4064" layer="1"/>
+<wire x1="43.688" y1="8.975" x2="43.664" y2="8.829" width="0.4064" layer="1"/>
 <wire x1="40.3921" y1="8.575" x2="42.611" y2="8.575" width="0.4064" layer="1"/>
-<wire x1="42.611" y1="8.575" x2="43.307" y2="9.017" width="0.4064" layer="1"/>
+<wire x1="42.611" y1="8.575" x2="43.561" y2="8.763" width="0.4064" layer="1"/>
 <wire x1="52.959" y1="9.652" x2="55.499" y2="9.652" width="0" layer="19" extent="1-1"/>
 </signal>
@@
 <contactref element="FB2" pad="1"/>
 <wire x1="33.716" y1="16.51" x2="33.716" y2="14.478" width="0.4064" layer="1"/>
-<wire x1="33.716" y1="14.478" x2="33.716" y2="12.7" width="0.4064" layer="1"/>
+<wire x1="33.716" y1="14.478" x2="33.716" y2="12.446" width="0.4064" layer="1"/>
 </signal>
 <signal name="N$5">
